File: electronics/arm_B.kicad_sch (KiCad schematic)
At the start: 26 parts, among them J13 EV3 B 4434 HOLD, J23 B SERVO G + S, U13 DRV8871DDAR, U23 SN74LVC2G17DBVR, U33 SN74AHCT1G125DBVR

Commit message: Integrate onboard RP2040 and drawing-based EV3 jacks on A1 PCB
Parts:
- J13: value EV3 B 4434 HOLD -> EV3 B PINMAP HOLD; footprint Quadcuber:EV3_4434_PROVISIONAL -> Quadcuber:EV3_UserDrawing_PINMAP_HOLD; MPN 4434 -> UNCONFIRMED user drawing; Manufacturer Adafruit (supplier brand) -> Unconfirmed (Coorle watermark)
- TP22, TP23, TP24, TP25: now left out of the parts list
Other:
- title: Quadcuber A0 / arm_B / ENGINEERING HOLD -> Quadcuber A1 / arm_B / ENGINEERING HOLD

Commit message: Correct audited power BOM and add bounded VM discharge protection
Parts:
- C161: MPN GRM32ER71E106KA12L -> GRM32DR71E106KA12L
- F13: footprint Quadcuber:Fuse_1812_4532Metric -> Quadcuber:Fuse_Bourns_MF_MSMF_Style2_1812; MPN MF-MSMF110-2 -> MF-MSMF110/16X-2
