File: electronics/flash_clock.kicad_sch (KiCad schematic)
At the start: 9 parts, among them U7 W25Q16JVSNIQ 2MiB, Y1 12MHz CL10pF

Commit message: Replace legacy Flash with production RV part and validate MicroPython boot2
Parts:
- U7: value W25Q16JVSNIQ 2MiB -> W25Q16RVCNJQ 2MiB; MPN W25Q16JVSNIQ -> W25Q16RVCNJQ
