File: electronics/quadcuber.kicad_pcb (KiCad board)
At the start: 4 copper layers, 144 x 112 mm, 159 parts, among them J1 9V regulated input, J10 EV3 R 4434 HOLD, J11 EV3 L 4434 HOLD, J12 EV3 F 4434 HOLD, J13 EV3 B 4434 HOLD, J2 UART GND TX RX, J20 R SERVO G + S, J21 L SERVO G + S, J22 F SERVO G + S, J23 B SERVO G + S, J3 RESET, Q1 CSD18540Q5B, U1 Pico H socketed, U10 DRV8871DDAR, U11 DRV8871DDAR, U12 DRV8871DDAR, U13 DRV8871DDAR, U2 TPS54302DDCR, U20 SN74LVC2G17DBVR, U21 SN74LVC2G17DBVR, U22 SN74LVC2G17DBVR, U23 SN74LVC2G17DBVR, U3 TPS54302DDCR, U30 SN74AHCT1G125DBVR, U31 SN74AHCT1G125DBVR, U32 SN74AHCT1G125DBVR, U33 SN74AHCT1G125DBVR, U4 LM74700QDBVRQ1

Commit message: Integrate onboard RP2040 and drawing-based EV3 jacks on A1 PCB
Parts:
- added C400: 100n, Quadcuber:C_0402_1005Metric, F.Cu at (61.0, 87.0)
- added C410: 100n, Quadcuber:C_0402_1005Metric, B.Cu at (65.6, 73.1)
- added C411: 100n, Quadcuber:C_0402_1005Metric, B.Cu at (66.8, 78.0)
- added C412: 100n, Quadcuber:C_0402_1005Metric, B.Cu at (69.0, 80.2)
- added C413: 100n, Quadcuber:C_0402_1005Metric, B.Cu at (73.7, 78.0)
- added C414: 100n, Quadcuber:C_0402_1005Metric, B.Cu at (76.5, 74.4)
- added C415: 100n, Quadcuber:C_0402_1005Metric, B.Cu at (73.9, 74.6)
- added C416: 100n, Quadcuber:C_0402_1005Metric, B.Cu at (71.7, 74.4)
- added C417: 100n, Quadcuber:C_0402_1005Metric, B.Cu at (72.3, 76.2)
- added C418: 100n, Quadcuber:C_0402_1005Metric, B.Cu at (70.6, 80.7)
- added C419: 100n, Quadcuber:C_0402_1005Metric, B.Cu at (70.3, 73.4)
- added C420: 1u, Quadcuber:C_0402_1005Metric, B.Cu at (74.3, 73.6)
- added C421: 1u, Quadcuber:C_0402_1005Metric, B.Cu at (73.1, 72.6)
- added C422: 4.7u/10V, Quadcuber:C_0805_2012Metric, F.Cu at (85.0, 70.0)
- added C423: 1u/16V, Quadcuber:C_0805_2012Metric, F.Cu at (87.0, 54.0)
- added C424: 100n, Quadcuber:C_0402_1005Metric, F.Cu at (64.0, 70.0)
- added C425: 15p, Quadcuber:C_0402_1005Metric, F.Cu at (66.7, 85.0)
- added C426: 15p, Quadcuber:C_0402_1005Metric, F.Cu at (73.2, 83.5)
- added C427: 100n, Quadcuber:C_0402_1005Metric, F.Cu at (74.0, 61.0)
- added D5: SS14 USB isolation, Quadcuber:D_SMA, B.Cu at (82.0, 63.0)
- added D7: USER LED GP25, Quadcuber:LED_0603_1608Metric, F.Cu at (78.0, 66.0)
- added F3: 0.5A USB PTC, Quadcuber:Fuse_1812_4532Metric, F.Cu at (82.0, 54.0)
- added J4: SWD VREF D G C, Quadcuber:PinHeader_1x04_P2.54mm_Vertical, F.Cu at (65.0, 105.0)
- added J5: USB-C data / BOOTSEL, Quadcuber:USB_C_Receptacle_GCT_USB4105-xx-A_16P_TopMnt_Horizontal, F.Cu at (70.0, 53.7)
- added R400: 10k, Quadcuber:R_0603_1608Metric, F.Cu at (58.0, 87.0)
- added R401: 5.1k, Quadcuber:R_0603_1608Metric, F.Cu at (62.0, 58.0)
- added R402: 5.1k, Quadcuber:R_0603_1608Metric, F.Cu at (78.0, 59.0)
- added R403: 27, Quadcuber:R_0402_1005Metric, F.Cu at (71.4, 71.0)
- added R404: 27, Quadcuber:R_0402_1005Metric, F.Cu at (70.4, 71.0)
- added R405: 100k, Quadcuber:R_0603_1608Metric, F.Cu at (84.0, 81.0)
- added R406: 100k, Quadcuber:R_0603_1608Metric, F.Cu at (84.0, 85.0)
- added R407: 10k, Quadcuber:R_0603_1608Metric, F.Cu at (63.0, 66.5)
- added R408: 1k, Quadcuber:R_0603_1608Metric, F.Cu at (57.0, 59.0)
- added R409: 1k, Quadcuber:R_0402_1005Metric, F.Cu at (74.0, 82.0)
- added R410: 1k, Quadcuber:R_0603_1608Metric, F.Cu at (75.0, 66.0)
- added S1: BOOTSEL, Quadcuber:SW_SPST_TL3342, F.Cu at (57.0, 63.0)
- added S2: RUN RESET, Quadcuber:SW_SPST_TL3342, F.Cu at (57.0, 93.0)
- added U5: TLV75533PDBVR, Quadcuber:SOT-23-5, F.Cu at (81.0, 72.0)
- added U6: USBLC6-2SC6, Quadcuber:SOT-23-6, F.Cu at (70.0, 62.0)
- added U7: W25Q16JVSNIQ 2MiB, Quadcuber:SOIC-8_3.9x4.9mm_P1.27mm, F.Cu at (60.0, 73.0)
- added Y1: 12MHz CL10pF, Quadcuber:Crystal_SMD_3225-4Pin_3.2x2.5mm, F.Cu at (70.0, 84.0)
- C1: value 10u/25V -> 1u/16V; footprint Quadcuber:C_1210_3225Metric -> Quadcuber:C_0805_2012Metric
- D2: value SS14 VSYS isolation -> SS14 external logic isolation
- J10: value EV3 R 4434 HOLD -> EV3 R PINMAP HOLD; footprint Quadcuber:EV3_4434_PROVISIONAL -> Quadcuber:EV3_UserDrawing_PINMAP_HOLD
- J11: value EV3 L 4434 HOLD -> EV3 L PINMAP HOLD; footprint Quadcuber:EV3_4434_PROVISIONAL -> Quadcuber:EV3_UserDrawing_PINMAP_HOLD
- J12: value EV3 F 4434 HOLD -> EV3 F PINMAP HOLD; footprint Quadcuber:EV3_4434_PROVISIONAL -> Quadcuber:EV3_UserDrawing_PINMAP_HOLD
- J13: value EV3 B 4434 HOLD -> EV3 B PINMAP HOLD; footprint Quadcuber:EV3_4434_PROVISIONAL -> Quadcuber:EV3_UserDrawing_PINMAP_HOLD
- U1: value Pico H socketed -> RP2040; footprint Quadcuber:Pico_H_Sockets -> Quadcuber:QFN-56-1EP_7x7mm_P0.4mm_EP3.2x3.2mm_ThermalVias
- moved U1 20.6 mm to (70.0, 77.0)
- moved C1 9.80 mm to (77.2, 70.0), turned to 180 degrees
- moved J10 4.12 mm to (66.0, 156.0), turned to 180 degrees
- moved J11 4.00 mm to (99.0, 156.0), turned to 180 degrees
- moved J12 4.00 mm to (133.0, 156.0), turned to 180 degrees
- moved J13 4.00 mm to (167.0, 156.0), turned to 180 degrees
Connections:
- U1 pad 1: GP0 -> 3V3
- U1 pad 10: GP7 -> 3V3
- U1 pad 13: GND -> GP10
- U1 pad 14: GP10 -> GP11
- U1 pad 15: GP11 -> GP12
- U1 pad 16: GP12 -> GP13
- U1 pad 17: GP13 -> GP14
- U1 pad 18: GND -> GP15
- U1 pad 19: GP14 -> GND
- U1 pad 2: GP1 -> GP0
- U1 pad 20: GP15 -> XIN
- U1 pad 21: GP16 -> XOUT
- U1 pad 22: GP17 -> 3V3
- U1 pad 23: GND -> 1V1
- U1 pad 24: GP18 -> SWCLK
- U1 pad 25: GP19 -> SWDIO
- U1 pad 26: GP20 -> RUN
- U1 pad 27: GP21 -> GP16
- U1 pad 28: GND -> GP17
- U1 pad 29: (no net) -> GP18
- U1 pad 3: GND -> GP1
- U1 pad 30: RUN -> GP19
- U1 pad 31: (no net) -> GP20
- U1 pad 32: (no net) -> GP21
- U1 pad 33: GND -> 3V3
- U1 pad 34: (no net) -> unconnected-(U1-GPIO22-Pad34)
- U1 pad 35: (no net) -> unconnected-(U1-GPIO23-Pad35)
- U1 pad 36: 3V3 -> GP24
- U1 pad 37: (no net) -> GP25
- U1 pad 38: GND -> unconnected-(U1-GPIO26-Pad38)
- U1 pad 39: VSYS -> unconnected-(U1-GPIO27-Pad39)
- U1 pad 40: (no net) -> unconnected-(U1-GPIO28-Pad40)
- U1 pad 8: GND -> GP6
- U1 pad 9: GP6 -> GP7
Routing:
- net USB_VBUS: track 0.00 -> 72.8 mm
- net R_ENC_A_RAW: track 22.4 -> 66.3 mm, vias 1 -> 0
- net QSPI_SS: track 0.00 -> 39.8 mm
- net SWDIO: track 0.00 -> 37.2 mm, vias 0 -> 3
- net GP16: track 87.8 -> 124.3 mm, vias 4 -> 3
- net GP21: track 180.3 -> 212.4 mm, vias 1 -> 0
- net RUN: track 29.6 -> 60.9 mm, vias 0 -> 7
- net GP17: track 95.2 -> 126.2 mm, vias 1 -> 4
- net SWCLK: track 0.00 -> 28.6 mm, vias 0 -> 2
- net GP9: track 109.4 -> 134.9 mm, vias 1 -> 2
- net GP20: track 141.3 -> 118.3 mm, vias 3 -> 6
- net GP19: track 141.1 -> 163.5 mm, vias 2 -> 4
- net GND: track 103.5 -> 124.3 mm, vias 96 -> 111
- net GP11: track 92.9 -> 113.5 mm, vias 1 -> 2
- net VSYS: track 133.7 -> 154.2 mm, vias 1 -> 4
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- added copper zone on In2.Cu, net 3V3
Other:
- board text added: "9V ONLY USB = LOGIC ONLY"
- board text added: "BOOT"
- board text added: "CLK"
- board text added: "EV3 PINMAP/CURRENT UNVERIFIED - DO NOT FABRICATE"
- board text added: "GP25"
- board text added: "IO"
- board text added: "QUADCUBER A1 / ENGINEERING HOLD"
- board text added: "RESET"
- board text added: "SWD"
- board text added: "USB"
- board text removed: "4434 JACK TAILS UNVERIFIED - DO NOT FABRICATE"
- board text removed: "9V ONLY USB = PICO ONLY"
- board text removed: "QUADCUBER A0 / ENGINEERING HOLD"

Commit message: Replace legacy Flash with production RV part and validate MicroPython boot2
Parts:
- U7: value W25Q16JVSNIQ 2MiB -> W25Q16RVCNJQ 2MiB
Changed lines of the file:
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@@
 			)
 		)
-		(property "Value" "W25Q16JVSNIQ 2MiB"
+		(property "Value" "W25Q16RVCNJQ 2MiB"
 			(at 0 3.4 0)
 			(layer "F.Fab")

Commit message: Correct audited power BOM and add bounded VM discharge protection
Parts:
- added R500: 300R 1W VM bleed, Quadcuber:R_2512_6332Metric, F.Cu at (175.0, 59.0)
- added R501: 300R 1W VM bleed, Quadcuber:R_2512_6332Metric, F.Cu at (175.0, 74.0)
- C422: value 4.7u/10V -> 4.7u/16V
- F1: value 8A 32V fuse -> 8A 24V time-lag fuse; footprint Quadcuber:Fuse_1206_3216Metric -> Quadcuber:Fuse_Littelfuse_407_1206
- F10, F11, F12, F13: footprint Quadcuber:Fuse_1812_4532Metric -> Quadcuber:Fuse_Bourns_MF_MSMF_Style2_1812
Routing:
- net VM: track 99.0 -> 102.6 mm, vias 43 -> 45
- net GND: track 124.3 -> 127.9 mm, vias 111 -> 113
