File: electronics/quadcuber.kicad_pcb (KiCad board)
At the start: 4 copper layers, 144 x 112 mm, 202 parts, among them J1 9V regulated input, J10 EV3 R PINMAP HOLD, J11 EV3 L PINMAP HOLD, J12 EV3 F PINMAP HOLD, J13 EV3 B PINMAP HOLD, J2 UART GND TX RX, J20 R SERVO G + S, J21 L SERVO G + S, J22 F SERVO G + S, J23 B SERVO G + S, J3 RESET, J4 SWD VREF D G C, J5 USB-C data / BOOTSEL, Q1 CSD18540Q5B, U1 RP2040, U10 DRV8871DDAR, U11 DRV8871DDAR, U12 DRV8871DDAR, U13 DRV8871DDAR, U2 TPS54302DDCR, U20 SN74LVC2G17DBVR, U21 SN74LVC2G17DBVR, U22 SN74LVC2G17DBVR, U23 SN74LVC2G17DBVR, U3 TPS54302DDCR, U30 SN74AHCT1G125DBVR, U31 SN74AHCT1G125DBVR, U32 SN74AHCT1G125DBVR, U33 SN74AHCT1G125DBVR, U4 LM74700QDBVRQ1, U5 TLV75533PDBVR, U6 USBLC6-2SC6, U7 W25Q16RVCNJQ 2MiB, Y1 12MHz CL10pF

Commit message: Correct A1 bootstrap routing and precision feedback with verified artifacts
Parts:
- removed R20, R30: 49.9, Quadcuber:R_0603_1608Metric
- moved C22 7.96 mm to (98.0, 91.9)
- moved C32 7.96 mm to (147.0, 91.9)
Connections:
- C22 pad 1: B1_BOOT_CAP -> B1_BOOT
- C32 pad 1: B2_BOOT_CAP -> B2_BOOT
Routing:
- net B2_SW: track 22.5 -> 10.9 mm
- net B1_SW: track 18.9 -> 10.9 mm
- net B2_BOOT: track 9.04 -> 3.29 mm, vias 2 -> 0
- net B1_BOOT: track 8.40 -> 3.29 mm
- net B2_BOOT_CAP: track 2.73 -> 0.00 mm
- net B1_BOOT_CAP: track 2.72 -> 0.00 mm
- net GND: track 127.9 -> 126.3 mm
- net B1_FB: track 17.6 -> 18.3 mm, vias 0 -> 2
