File: electronics-b1/quadcuber-b1.kicad_sch (KiCad schematic)
At the start: 66 parts, among them J1 9V DC 中心正, J10 舵机 R S+G, J11 EV3 R, J2 UART G TX RX, J20 舵机 L S+G, J21 EV3 L, J30 舵机 F S+G, J31 EV3 F, J40 舵机 B S+G, J41 EV3 B, Q1 IRF4905, U1 LM2596T-5.0, U10 DRV8871, U2 7805, U20 DRV8871, U3 Pico H, U30 DRV8871, U40 DRV8871

Commit message: B1 改为贴片为主：只保留插座和排针为通孔，并自带 3D 模型
- 用户要求元件尽量用贴片：P-MOS 改为 AO4407A（SOIC-8），舵机降压改为 LM2596S-5.0（TO-263-5），
  逻辑 5V 改为 AMS1117-5.0（SOT-223），二极管改为 SS34/SS14/SMBJ12A/BZT52C12，
  电阻电容改为 0805/2512，电解改为贴片铝电解，电感改为 12×12 贴片功率电感，保险丝改为 1206 慢断 8A。
  元件都放在顶面，便于热风枪手焊。
- 用户在 KiCad 3D 视图里看不到 Pico 和 DRV8871：KiCad Lite 不带标准 3D 库，DRV/EV3 的模型路径
  又指向 A1 工程。现把所用模型复制到 lib/3dmodels，统一用 ${KIPRJMOD} 引用。
- 布线：VM 主干改到底层 x=36 竖线 + y=57.4 横条（只覆盖四颗 DRV），两端留出底层通道；
  每个贴片接地脚就近打孔；铺铜后在至少一面是主地铜的位置打缝合过孔；KiCad 间距规则比
  freerouting 少 0.05mm 余量，消除 Pico 异形焊盘的近似误差。
- 结果：DRC 0 错误、0 未连通（26 条警告：丝印重叠和主干端点）；test_b1 5/5 通过；
  A1 及其首板包未改动。

Co-Authored-By: Claude Opus 5.5 <noreply@anthropic.com>
Parts:
- C1, C2: footprint B1:CP_Radial_D10.0mm_P5.00mm -> B1:CP_Elec_10x10.5
- C10, C20, C30, C40, C7: footprint B1:C_Disc_D3.0mm_W1.6mm_P2.50mm -> B1:C_0805_2012Metric_Pad1.18x1.45mm_HandSolder
- C11, C21, C31, C41: footprint B1:CP_Radial_D6.3mm_P2.50mm -> B1:CP_Elec_6.3x7.7
- C3, C4: footprint B1:CP_Radial_D8.0mm_P3.50mm -> B1:CP_Elec_8x10.5
- C5: value 0.33u -> 10u/25V; footprint B1:C_Disc_D3.0mm_W1.6mm_P2.50mm -> B1:C_0805_2012Metric_Pad1.18x1.45mm_HandSolder
- C6: value 10u/16V -> 22u/16V; footprint B1:CP_Radial_D5.0mm_P2.00mm -> B1:C_0805_2012Metric_Pad1.18x1.45mm_HandSolder
- D1: value P6KE15A -> SMBJ12A; footprint B1:D_DO-15_P10.16mm_Horizontal -> B1:D_SMB_Handsoldering
- D2: value 1N5822 -> SS34; footprint B1:D_DO-201AD_P15.24mm_Horizontal -> B1:D_SMA_Handsoldering
- D3: value 1N5819 -> SS14; footprint B1:D_DO-41_SOD81_P10.16mm_Horizontal -> B1:D_SMA_Handsoldering
- DZ1: footprint B1:D_DO-41_SOD81_P10.16mm_Horizontal -> B1:D_SOD-123
- F1: value PTC 5A -> 8A 慢断; footprint B1:Fuse_PTC_Radial_P5.10mm -> B1:Fuse_1206_3216Metric_Pad1.42x1.75mm_HandSolder
- L1: footprint B1:L_Radial_D10.0mm_P5.00mm_Fastron_07M -> B1:L_12x12mm_H8mm
- Q1: value IRF4905 -> AO4407A; footprint B1:TO-220-3_Vertical -> B1:SOIC-8_3.9x4.9mm_P1.27mm
- R1, R10, R20, R30, R40: footprint B1:R_Axial_DIN0207_L6.3mm_D2.5mm_P7.62mm_Horizontal -> B1:R_0805_2012Metric_Pad1.20x1.40mm_HandSolder
- R11, R12, R13, R14, R15, R21, R22, R23, R24, R25, R31, R32, R33, R34, R35, R41, R42, R43, R44, R45: footprint B1:R_Axial_DIN0207_L6.3mm_D2.5mm_P2.54mm_Vertical -> B1:R_0805_2012Metric_Pad1.20x1.40mm_HandSolder
- R2, R3: footprint B1:R_Axial_DIN0414_L11.9mm_D4.5mm_P5.08mm_Vertical -> B1:R_2512_6332Metric_Pad1.40x3.35mm_HandSolder
- U1: value LM2596T-5.0 -> LM2596S-5.0; footprint B1:TO-220-5_P3.4x3.7mm_StaggerOdd_Lead3.8mm_Vertical -> B1:TO-263-5_TabPin3
- U2: value 7805 -> AMS1117-5.0; footprint B1:TO-220-3_Vertical -> B1:SOT-223-3_TabPin2
Connections:
- net 5V_LOGIC: now also U2.2; no longer U2.3
- net GATE: now also Q1.4; no longer Q1.1
- net GND: now also U2.1; no longer U2.2
- net VIN_F: now also Q1.5, Q1.6, Q1.7, Q1.8; no longer Q1.2
- net VM: now also Q1.1, Q1.2, U2.3; no longer U2.1
